File: ZX80_Gaming_Keyboard/ZX80_Gaming_Keyboard.kicad_pcb (KiCad board)
At the start: 2 copper layers, 276 x 89 mm, 52 parts, among them J1 KB1, J2 KB2, J3 0_SPACE, SW1 1, SW10 0, SW11 Q, SW12 W, SW13 E, SW14 R, SW15 T, SW16 Y, SW17 U, SW18 I, SW19 O, SW2 2, SW20 P, SW21 A, SW22 S, SW23 D, SW24 F, SW25 G, SW26 H, SW27 J, SW28 K, SW29 L, SW3 3, SW30 NL, SW31 SHIFT, SW32 Z, SW33 X, SW34 C, SW35 V, SW36 B, SW37 N, SW38 M, SW39 DOT, SW4 4, SW40 SPACE, SW41 LEFT, SW42 DOWN, SW43 UP, SW44 RIGHT, SW45 RUBOUT, SW5 5, SW6 6, SW7 7, SW8 8, SW9 9

Commit message: Finalised keyboard design for testing
Other:
- board text added: "Rev. A"
Changed lines of the file:
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@@
+		)
+	)
+	(gr_text "Rev. A"
+		(at 87.378594 186.265581 0)
+		(layer "B.SilkS")
+		(effects
+			(font
+				(size 1.5 1.5)
+				(thickness 0.3)
+				(bold yes)
+			)
+			(justify left bottom mirror)
 		)
 	)
