File: ZX80_Gaming_Keyboard/ZX80_Gaming_Keyboard.kicad_pcb (KiCad board)
At the start: 2 copper layers, 276 x 89 mm, 52 parts, among them J1 KB1, J2 KB2, J3 0_SPACE, SW1 1, SW10 0, SW11 Q, SW12 W, SW13 E, SW14 R, SW15 T, SW16 Y, SW17 U, SW18 I, SW19 O, SW2 2, SW20 P, SW21 A, SW22 S, SW23 D, SW24 F, SW25 G, SW26 H, SW27 J, SW28 K, SW29 L, SW3 3, SW30 NL, SW31 SHIFT, SW32 Z, SW33 X, SW34 C, SW35 V, SW36 B, SW37 N, SW38 M, SW39 DOT, SW4 4, SW40 SPACE, SW41 LEFT, SW42 DOWN, SW43 UP, SW44 RIGHT, SW45 RUBOUT, SW5 5, SW6 6, SW7 7, SW8 8, SW9 9

Commit message: Revised PCB layout correcting errors
Parts:
- added D1: 1N4148, Diode_THT:D_DO-35_SOD27_P7.62mm_Horizontal, F.Cu at (306.1, 116.3)
- added D2: 1N4148, Diode_THT:D_DO-35_SOD27_P7.62mm_Horizontal, F.Cu at (306.1, 121.4)
- added S1: 76STD01T, Button_Switch_THT:76STD01T, F.Cu at (345.5, 143.0)
- J3: value 0_SPACE -> SPACE_ZERO
- moved J3 57.3 mm to (349.3, 159.5), turned to 180 degrees
- moved J2 50.4 mm to (241.7, 104.6)
- moved J1 46.6 mm to (226.5, 104.6)
- moved SW45 16.5 mm to (329.0, 115.0)
Connections:
- net ~{A14} renamed A14
- net ~{A15} renamed A15
- J2 pad 6: A12 -> A8
- SW31 pad 2: A12 -> A8
- SW32 pad 2: A12 -> A8
- SW33 pad 2: A12 -> A8
- SW34 pad 2: A12 -> A8
- SW35 pad 2: A12 -> A8
- SW42 pad 1: COL1 -> CUR_DOWN
- SW43 pad 1: COL2 -> CUR_UP
- SW45 pad 2: A12 -> Net-(D1-A)
Routing:
- net A8: track 0.00 -> 285.3 mm, vias 0 -> 2
- net A12: track 388.8 -> 247.7 mm
- net CUR_DOWN: track 0.00 -> 64.4 mm
- net A9: track 241.2 -> 190.0 mm
- net A10: track 222.1 -> 172.5 mm
- net COL3: track 385.5 -> 347.3 mm, vias 1 -> 0
- net CUR_UP: track 0.00 -> 35.8 mm, vias 0 -> 1
- net A15: track 205.8 -> 239.4 mm
- net COL1: track 328.1 -> 359.8 mm
- net Net-(J3-Pin_2): track 129.0 -> 103.4 mm
- net A13: track 132.6 -> 112.8 mm, vias 1 -> 0
- net A14: track 163.7 -> 143.9 mm, vias 1 -> 0
- net Net-(D1-A): track 0.00 -> 14.5 mm
- net COL4: track 305.2 -> 291.6 mm, vias 0 -> 2
- net A11: track 272.4 -> 283.0 mm, vias 1 -> 2
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Other:
- board text added: "A11 A10 A12 A9 A13 A8 A14 A15"
- board text added: "ACE ZX"
- board text added: "ACE/ZX switches cursor UP/DOWN keys ZX: [6] = DOWN [7] = UP ACE: [6] = UP [7] = DOWN SPACE/0 changes [SPACE] to [0] for games like KONG"
- board text added: "BRETT'S ZX/ACE GAMING KEYBOARD"
- board text added: "COL1 COL2 COL3 COL4 COL5"
- board text added: "Rev. B"
- board text added: "SPACE 0"
- board text removed: "0"
- board text removed: "BRETT'S MINSTREL GAMING KEYBOARD"
- board text removed: "Rev. A"
- board text removed: "SPACE"

Commit message: Revised ZX/ACE switch
Parts:
- removed S1: 76STD01T, Button_Switch_THT:76STD01T
- added J4: ZX_ACE, Connector_PinHeader_2.54mm:PinHeader_2x02_P2.54mm_Vertical, F.Cu at (346.8, 146.8)
- moved SW45 35.5 mm to (293.5, 115.0)
- moved D2 5.39 mm to (309.9, 117.6), turned to -90 degrees
- moved D1 1.80 mm to (304.8, 117.6), turned to -90 degrees
Routing:
- net COL5: track 377.3 -> 341.6 mm
- net COL1: track 359.8 -> 338.8 mm
- net Net-(D1-A): track 14.5 -> 27.4 mm
- net A15: track 239.4 -> 227.9 mm
- net CUR_DOWN: track 64.4 -> 53.8 mm, vias 0 -> 1
- net A12: track 247.7 -> 256.2 mm
- net A13: track 112.8 -> 121.1 mm
- net A8: track 285.3 -> 290.5 mm
- net A11: track 283.0 -> 278.2 mm
- net Net-(J3-Pin_2): track 103.4 -> 99.0 mm
- net CUR_UP: track 35.8 -> 39.9 mm, vias 1 -> 0
- net COL3: track 347.3 -> 350.6 mm, vias 0 -> 1
- net A14: track 143.9 -> 142.5 mm
Other:
- board text added: "ACE"
- board text added: "ZX"
- board text removed: "ACE ZX"

Commit message: Initial Rev. C changes
Parts:
- removed the D1 at (304.8, 117.6)
- moved J3 55.2 mm to (343.3, 104.6), turned to 90 degrees
- moved J4 44.3 mm to (333.2, 104.6)
- moved D1 36.3 mm to (276.0, 104.6), turned to 0 degrees
- moved J2 2.54 mm to (244.3, 104.6)
- renumbered D2 to D1
Connections:
- D1 pad 2: Net-(D1-A) -> A8
- SW45 pad 2: Net-(D1-A) -> A8
Routing:
- net Net-(J3-Pin_2): track 99.0 -> 143.2 mm
- net A8: track 290.5 -> 255.1 mm, vias 2 -> 1
- net Net-(D1-A): track 27.4 -> 0.00 mm
- net CUR_DOWN: track 53.8 -> 73.6 mm, vias 1 -> 0
- net CUR_UP: track 39.9 -> 59.6 mm
- net COL1: track 338.8 -> 357.5 mm
- net COL2: track 338.7 -> 327.4 mm
- net A13: track 121.1 -> 112.2 mm
- net A12: track 256.2 -> 264.4 mm, vias 0 -> 1
- net A11: track 278.2 -> 270.0 mm
- net A14: track 142.5 -> 147.8 mm
- net COL5: track 341.6 -> 346.1 mm, vias 0 -> 1
- net A15: track 227.9 -> 223.6 mm
- net COL4: track 291.5 -> 287.6 mm
- net COL3: track 350.6 -> 354.4 mm, vias 1 -> 0
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Other:
- board text added: "ACE/ZX switches cursor UP/DOWN keys ZX: [6] = DOWN [7] = UP ACE: [6] = UP [7] = DOWN SPACE/0 changes [SPACE] to [0]"
- board text added: "Rev. C"
- board text removed: "ACE/ZX switches cursor UP/DOWN keys ZX: [6] = DOWN [7] = UP ACE: [6] = UP [7] = DOWN SPACE/0 changes [SPACE] to [0] for games like KONG"
- board text removed: "Rev. B"
