File: Z88_Mechanical_Keyboard/Z88_Mechanical_Keyboard.kicad_pcb (KiCad board)
At the start: 2 copper layers, 295 x 117 mm, 66 parts, among them SW1 SHIFT_RH, SW10 SHIFT_LH, SW11 SPACE, SW12 LEFT, SW13 RIGHT, SW14 DOWN, SW15 UP, SW16 ENTER, SW17 ESC, SW18 TAB, SW19 1, SW2 HELP, SW20 2, SW21 3, SW22 4, SW23 5, SW24 6, SW25 INDEX, SW26 DIAMOND, SW27 Q, SW28 W, SW29 E, SW3 [, SW30 R, SW31 T, SW32 Y, SW33 CAPS_LOCK, SW34 MENU, SW35 A, SW36 S, SW37 D, SW38 F, SW39 G, SW4 ], SW40 H, SW41 DOT, SW42 COMMA, SW43 Z, SW44 X, SW45 C, SW46 V, SW47 B, SW48 N, SW49 /, SW5 UNDERSCORE, SW50 SEMICOLON, SW51 L, SW52 M, SW53 K, SW54 J, SW55 U, SW56 7, SW57 £, SW58 DOUBLE_QUOTE, SW59 0, SW6 =, SW60 P, SW61 9, SW62 O, SW63 I, SW64 8, SW7 \, SW8 DELETE, SW9 SQUARE

Commit message: Progress commit
Parts:
- moved SW1 37.9 mm to (312.5, 168.7)
- moved SW41 37.9 mm to (265.0, 168.7)
- moved SW47 37.9 mm to (188.7, 168.7)
- moved SW49 37.9 mm to (284.0, 168.7)
- moved SW10 37.9 mm to (83.9, 168.7)
- moved SW11 37.9 mm to (207.8, 187.7)
- moved SW42 37.9 mm to (245.9, 168.7)
- moved SW43 37.9 mm to (112.5, 168.7)
- moved SW44 37.9 mm to (131.6, 168.7)
- moved SW45 37.9 mm to (150.6, 168.7)
- moved SW46 37.9 mm to (169.7, 168.7)
- moved SW48 37.9 mm to (207.8, 168.7)
- moved SW52 37.9 mm to (226.8, 168.7)
- moved SW16 37.9 mm to (338.8, 140.0)
- moved SW50 37.9 mm to (279.2, 149.6)
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Routing:
- net COL4: track 65.1 -> 507.6 mm, vias 0 -> 4
- net ROW0: track 0.00 -> 416.3 mm, vias 0 -> 2
- net COL3: track 65.1 -> 455.1 mm, vias 0 -> 7
- net ROW1: track 0.00 -> 385.3 mm
- net COL0: track 135.9 -> 489.1 mm, vias 0 -> 2
- net ROW3: track 0.00 -> 331.3 mm, vias 0 -> 1
- net COL5: track 65.1 -> 393.8 mm, vias 0 -> 4
- net COL2: track 65.1 -> 391.7 mm, vias 0 -> 6
- net COL6: track 65.1 -> 364.8 mm, vias 0 -> 3
- net COL1: track 84.4 -> 383.4 mm, vias 0 -> 2
- net COL7: track 0.00 -> 298.8 mm, vias 0 -> 2
- net ROW5: track 0.00 -> 284.8 mm, vias 0 -> 2
- net ROW4: track 0.00 -> 268.4 mm, vias 0 -> 3
- net ROW6: track 0.00 -> 244.1 mm, vias 0 -> 2
- net ROW7: track 0.00 -> 224.7 mm
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Other:
- board size 295 x 117 mm -> 291 x 115 mm
- board text added: "Cambridge Computer Z88"

Commit message: Added 3D models
Parts:
- SK6, SK7: footprint Connector_PinHeader_2.54mm:PinHeader_1x08_P2.54mm_Horizontal -> Clueless_Engineer:55203148
- moved SK6 21.9 mm to (273.7, 95.0), turned to 0 degrees
- moved SK7 19.9 mm to (300.7, 95.0), turned to 0 degrees
Routing:
- net COL4: track 507.6 -> 0.00 mm, vias 4 -> 0
- net COL0: track 489.1 -> 0.00 mm, vias 2 -> 0
- net COL3: track 455.1 -> 0.00 mm, vias 7 -> 0
- net ROW0: track 416.3 -> 0.00 mm, vias 2 -> 0
- net COL5: track 393.8 -> 0.00 mm, vias 4 -> 0
- net COL2: track 391.7 -> 0.00 mm, vias 6 -> 0
- net ROW1: track 385.3 -> 0.00 mm
- net COL1: track 383.4 -> 0.00 mm, vias 2 -> 0
- net COL6: track 364.8 -> 0.00 mm, vias 3 -> 0
- net ROW3: track 331.3 -> 0.00 mm, vias 1 -> 0
- net ROW2: track 323.8 -> 0.00 mm, vias 1 -> 0
- net COL7: track 298.8 -> 0.00 mm, vias 2 -> 0
- net ROW5: track 284.8 -> 0.00 mm, vias 2 -> 0
- net ROW4: track 268.4 -> 0.00 mm, vias 3 -> 0
- net ROW6: track 244.1 -> 0.00 mm, vias 2 -> 0
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