File: Z88_Mechanical_Keyboard/Z88_Mechanical_Keyboard.kicad_pcb (KiCad board)
At the start: 2 copper layers, 291 x 115 mm, 66 parts, among them SW1 SHIFT_RH, SW10 SHIFT_LH, SW11 SPACE, SW12 LEFT, SW13 RIGHT, SW14 DOWN, SW15 UP, SW16 ENTER, SW17 ESC, SW18 TAB, SW19 1, SW2 HELP, SW20 2, SW21 3, SW22 4, SW23 5, SW24 6, SW25 INDEX, SW26 DIAMOND, SW27 Q, SW28 W, SW29 E, SW3 [, SW30 R, SW31 T, SW32 Y, SW33 CAPS_LOCK, SW34 MENU, SW35 A, SW36 S, SW37 D, SW38 F, SW39 G, SW4 ], SW40 H, SW41 DOT, SW42 COMMA, SW43 Z, SW44 X, SW45 C, SW46 V, SW47 B, SW48 N, SW49 /, SW5 UNDERSCORE, SW50 SEMICOLON, SW51 L, SW52 M, SW53 K, SW54 J, SW55 U, SW56 7, SW57 £, SW58 DOUBLE_QUOTE, SW59 0, SW6 =, SW60 P, SW61 9, SW62 O, SW63 I, SW64 8, SW7 \, SW8 DELETE, SW9 SQUARE

Commit message: Keyboard layout changes
Parts:
- added H1: MountingHole, MountingHole:MountingHole_3.2mm_M3, F.Cu at (67.5, 93.0)
- added H2: MountingHole, MountingHole:MountingHole_3.2mm_M3, F.Cu at (348.5, 93.0)
- SK6, SK7: moved to F.Cu
- SW19: value 1 -> ONE
- SW49: value / -> /FORWSLASH/
- SW57: value £ -> GBP
- SW59: value 0 -> ZERO
- SW6: value = -> EQUALS
- SW7: value \ -> \BACKSLASH\
- moved SW11 7.17 mm to (200.7, 187.7)
- moved SW33 7.05 mm to (276.9, 187.7)
- moved SK7 4.68 mm to (296.5, 97.0)
- moved SK6 3.80 mm to (270.5, 97.0)
Other:
- board size 291 x 115 mm -> 289 x 110 mm
- board text added: "Cambridge Computer Z88 Mechanical Keyboard Brett Hallen, Jul 2025 Port Macquarie, Australia"
