File: Z88_Mechanical_Keyboard/Z88_Mechanical_Keyboard.kicad_pcb (KiCad board)
At the start: 2 copper layers, 289 x 110 mm, 72 parts, among them SW1 SHIFT_RH, SW10 SHIFT_LH, SW11 SPACE, SW12 LEFT, SW13 RIGHT, SW14 DOWN, SW15 UP, SW16 ENTER, SW17 ESC, SW18 TAB, SW19 ONE, SW2 HELP, SW20 2, SW21 3, SW22 4, SW23 5, SW24 6, SW25 INDEX, SW26 DIAMOND, SW27 Q, SW28 W, SW29 E, SW3 [, SW30 R, SW31 T, SW32 Y, SW33 CAPS_LOCK, SW34 MENU, SW35 A, SW36 S, SW37 D, SW38 F, SW39 G, SW4 ], SW40 H, SW41 DOT, SW42 COMMA, SW43 Z, SW44 X, SW45 C, SW46 V, SW47 B, SW48 N, SW49 /FORWSLASH/, SW5 UNDERSCORE, SW50 SEMICOLON, SW51 L, SW52 M, SW53 K, SW54 J, SW55 U, SW56 7, SW57 GBP, SW58 DOUBLE_QUOTE, SW59 ZERO, SW6 EQUALS, SW60 P, SW61 9, SW62 O, SW63 I, SW64 8, SW7 \BACKSLASH\, SW8 DELETE, SW9 SQUARE

Commit message: Swapped DOWN/RIGHT cursors (thanks Alex Q)
Parts:
- moved SW33 57.2 mm to (341.1, 187.7)
- moved SW14 38.1 mm to (303.0, 187.7)
- moved SW15 38.1 mm to (303.0, 168.7)
- moved KB2 19.1 mm to (331.7, 168.7)
- moved SW1 19.1 mm to (331.7, 168.7)
- moved SW12 19.1 mm to (283.9, 187.7)
- moved SW13 0.06 mm to (322.1, 187.7)
Routing:
- net COL0: track 371.1 -> 0.00 mm
- net ROW1: track 325.7 -> 0.00 mm
- net ROW0: track 316.2 -> 0.00 mm
- net COL6: track 295.0 -> 0.00 mm, vias 1 -> 0
- net COL4: track 256.6 -> 0.00 mm
- net ROW3: track 171.0 -> 0.00 mm
- net COL2: track 168.1 -> 0.00 mm
- net ROW5: track 163.0 -> 0.00 mm
- net ROW7: track 155.4 -> 0.00 mm
- net ROW2: track 148.7 -> 0.00 mm
- net ROW4: track 145.5 -> 0.00 mm
- net COL7: track 139.6 -> 0.00 mm
- net ROW6: track 125.8 -> 0.00 mm
- net COL1: track 84.4 -> 0.00 mm
- net COL3: track 65.1 -> 0.00 mm
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
Commit message: Routing completed
Routing:
- net ROW5: track 0.00 -> 464.1 mm, vias 0 -> 1
- net COL0: track 0.00 -> 463.5 mm, vias 0 -> 1
- net ROW1: track 0.00 -> 438.9 mm
- net ROW0: track 0.00 -> 382.7 mm
- net COL3: track 0.00 -> 381.7 mm, vias 0 -> 3
- net ROW4: track 0.00 -> 379.9 mm, vias 0 -> 1
- net COL4: track 0.00 -> 371.0 mm, vias 0 -> 3
- net COL1: track 0.00 -> 368.7 mm, vias 0 -> 1
- net COL2: track 0.00 -> 364.5 mm, vias 0 -> 1
- net COL5: track 0.00 -> 335.8 mm, vias 0 -> 1
- net ROW3: track 0.00 -> 331.7 mm, vias 0 -> 1
- net COL6: track 0.00 -> 327.9 mm, vias 0 -> 1
- net COL7: track 0.00 -> 272.1 mm
- net ROW2: track 0.00 -> 271.3 mm
- net ROW6: track 0.00 -> 254.9 mm, vias 0 -> 2
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Other:
- outline, holes or cut-outs redrawn
- board text added: "Rev. A"
