File: Z88_Mechanical_Keyboard/7u_SPACE/Z88_Mechanical_Keyboard.kicad_pcb (KiCad board)
At the start: 2 copper layers, 289 x 110 mm, 68 parts, among them SW1 SHIFT_RH, SW10 SHIFT_LH, SW11 SPACE, SW12 LEFT, SW13 RIGHT, SW14 DOWN, SW15 UP, SW16 ENTER, SW17 ESC, SW18 TAB, SW19 ONE, SW2 HELP, SW20 2, SW21 3, SW22 4, SW23 5, SW24 6, SW25 INDEX, SW26 DIAMOND, SW27 Q, SW28 W, SW29 E, SW3 [, SW30 R, SW31 T, SW32 Y, SW33 CAPS_LOCK, SW34 MENU, SW35 A, SW36 S, SW37 D, SW38 F, SW39 G, SW4 ], SW40 H, SW41 DOT, SW42 COMMA, SW43 Z, SW44 X, SW45 C, SW46 V, SW47 B, SW48 N, SW49 /FORWSLASH/, SW5 UNDERSCORE, SW50 SEMICOLON, SW51 L, SW52 M, SW53 K, SW54 J, SW55 U, SW56 7, SW57 GBP, SW58 DOUBLE_QUOTE, SW59 ZERO, SW6 EQUALS, SW60 P, SW61 9, SW62 O, SW63 I, SW64 8, SW7 \BACKSLASH\, SW8 DELETE, SW9 SQUARE

Commit message: Added T-cursor layout
Parts:
- added KB1: ~, PCM_Mounting_Keyboard_Stabilizer:Stabilizer_Cherry_MX_2.00u, F.Cu at (83.9, 168.7)
- added KB2: , PCM_Mounting_Keyboard_Stabilizer:Stabilizer_Cherry_MX_2.00u, F.Cu at (312.5, 168.7)
- added KB3: ~, PCM_Mounting_Keyboard_Stabilizer:Stabilizer_Cherry_MX_2.00u, F.Cu at (338.7, 140.0)
- added KB4: ~, PCM_Mounting_Keyboard_Stabilizer:Stabilizer_Cherry_MX_7.00u, F.Cu at (207.5, 187.7)
Routing:
- net COL0: track 0.00 -> 371.1 mm
- net ROW1: track 0.00 -> 325.7 mm
- net ROW0: track 0.00 -> 316.2 mm
- net COL6: track 0.00 -> 295.0 mm, vias 0 -> 1
- net COL4: track 0.00 -> 256.6 mm
- net ROW3: track 0.00 -> 171.0 mm
- net COL2: track 0.00 -> 168.1 mm
- net ROW5: track 0.00 -> 163.0 mm
- net ROW7: track 0.00 -> 155.4 mm
- net ROW2: track 0.00 -> 148.7 mm
- net ROW4: track 0.00 -> 145.5 mm
- net COL7: track 0.00 -> 139.6 mm
- net ROW6: track 0.00 -> 125.8 mm
- net COL1: track 0.00 -> 84.4 mm
- net COL3: track 0.00 -> 65.1 mm
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Other:
- board text added: "7u SPACE"
