File: Z88_Mechanical_Keyboard/T_CURSOR/Z88_Mechanical_Keyboard.kicad_pcb (KiCad board)
At the start: 2 copper layers, 289 x 110 mm, 71 parts, among them SW1 SHIFT_RH, SW10 SHIFT_LH, SW11 SPACE, SW12 LEFT, SW13 RIGHT, SW14 DOWN, SW15 UP, SW16 ENTER, SW17 ESC, SW18 TAB, SW19 ONE, SW2 HELP, SW20 2, SW21 3, SW22 4, SW23 5, SW24 6, SW25 INDEX, SW26 DIAMOND, SW27 Q, SW28 W, SW29 E, SW3 [, SW30 R, SW31 T, SW32 Y, SW33 CAPS_LOCK, SW34 MENU, SW35 A, SW36 S, SW37 D, SW38 F, SW39 G, SW4 ], SW40 H, SW41 DOT, SW42 COMMA, SW43 Z, SW44 X, SW45 C, SW46 V, SW47 B, SW48 N, SW49 /FORWSLASH/, SW5 UNDERSCORE, SW50 SEMICOLON, SW51 L, SW52 M, SW53 K, SW54 J, SW55 U, SW56 7, SW57 GBP, SW58 DOUBLE_QUOTE, SW59 ZERO, SW6 EQUALS, SW60 P, SW61 9, SW62 O, SW63 I, SW64 8, SW7 \BACKSLASH\, SW8 DELETE, SW9 SQUARE

Commit message: Modified T-cursor layout
Parts:
- added KB2: , PCM_Mounting_Keyboard_Stabilizer:Stabilizer_Cherry_MX_2.00u, F.Cu at (331.7, 168.7)
- moved SW33 57.2 mm to (341.1, 187.7)
- moved SW1 28.7 mm to (331.7, 168.7)
- moved SW13 19.1 mm to (303.0, 187.7)
- moved SW12 19.1 mm to (283.9, 187.7)
- moved SW14 19.1 mm to (322.0, 187.7)
- moved SW15 19.0 mm to (303.0, 168.7)

Commit message: Routing completed
Parts:
- moved SW13 19.1 mm to (322.1, 187.7)
- moved SW14 19.0 mm to (303.0, 187.7)
Routing:
- net ROW5: track 0.00 -> 464.1 mm, vias 0 -> 1
- net COL0: track 0.00 -> 463.5 mm, vias 0 -> 1
- net ROW1: track 0.00 -> 438.9 mm
- net ROW0: track 0.00 -> 382.7 mm
- net COL3: track 0.00 -> 381.7 mm, vias 0 -> 3
- net ROW4: track 0.00 -> 379.9 mm, vias 0 -> 1
- net COL4: track 0.00 -> 371.0 mm, vias 0 -> 3
- net COL1: track 0.00 -> 368.7 mm, vias 0 -> 1
- net COL2: track 0.00 -> 364.5 mm, vias 0 -> 1
- net COL5: track 0.00 -> 335.8 mm, vias 0 -> 1
- net ROW3: track 0.00 -> 331.7 mm, vias 0 -> 1
- net COL6: track 0.00 -> 327.9 mm, vias 0 -> 1
- net COL7: track 0.00 -> 272.1 mm
- net ROW2: track 0.00 -> 271.3 mm
- net ROW6: track 0.00 -> 254.9 mm, vias 0 -> 2
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Other:
- outline, holes or cut-outs redrawn
- board text added: "Rev. A"

Commit message: Final tweaks before test fabrication
Parts:
- KB1: value ~ -> SHIFT_LH
- KB2: value (none) -> SHIFT_RH
- KB3: value ~ -> ENTER
- KB4: value ~ -> SPACE_BAR
- SW12: value LEFT -> VASEN
- SW13: value RIGHT -> OIKEIN
- SW14: value DOWN -> ALAS
- SW15: value UP -> YLÖS
- SW19: value ONE -> YKSI
- SW2: value HELP -> APUA!
- SW20: value 2 -> KAKSI
- SW21: value 3 -> KOLME
- SW22: value 4 -> NELJÄ
- SW23: value 5 -> VIISI
- SW24: value 6 -> KUUSI
- SW56: value 7 -> SEITSEMÄN
- SW59: value ZERO -> NOLLA
- SW61: value 9 -> YHDEKSÄN
- SW64: value 8 -> KAHDEKSAN
- moved H1 28.3 mm to (95.5, 97.0)
- moved H2 11.7 mm to (337.5, 97.0)
Routing:
- net COL1: track 368.7 -> 511.2 mm
- net COL3: track 381.7 -> 373.2 mm, vias 3 -> 2
- net ROW0: track 382.7 -> 388.3 mm
- net ROW4: track 379.9 -> 383.4 mm
- net COL4: track 371.0 -> 373.2 mm, vias 3 -> 2
- net COL6: track 327.9 -> 330.1 mm, vias 1 -> 2
- net COL5: track 335.8 -> 336.9 mm
- net ROW1: track 438.9 -> 440.0 mm
- net COL2: track 364.5 -> 365.3 mm
- net ROW3: track 331.7 -> 332.3 mm
Other:
- board text added: "A14 A15 A13 A12 A11 A10 A9 A8"
- board text added: "Cambridge Computer Z88 Mechanical Keyboard Brett Hallen, Jul 2025 Port Macquarie, Australia WWW.YOUTUBE.COM/@BRFFF"
- board text added: "D5 D4 D3 D1 D7 D0 D6 D2"
- board text removed: "Cambridge Computer Z88 Mechanical Keyboard Brett Hallen, Jul 2025 Port Macquarie, Australia"
