File: Z88_Mechanical_Keyboard/Rev_A/Z88_Mechanical_Keyboard_Rev_A.kicad_pcb (KiCad board)
At the start: 2 copper layers, 289 x 110 mm, 72 parts, among them SW1 SHIFT_RH, SW10 SHIFT_LH, SW11 SPACE, SW12 VASEN, SW13 OIKEIN, SW14 ALAS, SW15 YLÖS, SW16 ENTER, SW17 ESC, SW18 TAB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

Commit message: Archiving Rev. A design
Parts:
- added G***: LOGO, LOGO, F.Cu at (-255.5, -220.3)
Other:
- board text added: "ISO ENTER"
- board text added: "Sponsored by"
