File: Z88_Mechanical_Keyboard/Rev_B/Z88_Mechanical_Keyboard_Rev_B.kicad_pcb (KiCad board)
At the start: 2 copper layers, 289 x 110 mm, 70 parts, among them SW1 SHIFT_RH, SW10 SHIFT_LH, SW11 SPACE, SW12 VASEN, SW13 OIKEIN, SW14 ALAS, SW15 YLÖS, SW16 ENTER, SW17 ESC, SW18 TAB, SW19 YKSI, SW2 APUA!, SW20 KAKSI, SW21 KOLME, SW22 NELJÄ, SW23 VIISI, SW24 KUUSI, SW25 INDEX, SW26 DIAMOND, SW27 Q, SW28 W, SW29 E, SW3 [, SW30 R, SW31 T, SW32 Y, SW33 CAPS_LOCK, SW34 MENU, SW35 A, SW36 S, SW37 D, SW38 F, SW39 G, SW4 ], SW40 H, SW41 DOT, SW42 COMMA, SW43 Z, SW44 X, SW45 C, SW46 V, SW47 B, SW48 N, SW49 /FORWSLASH/, SW5 UNDERSCORE, SW50 SEMICOLON, SW51 L, SW52 M, SW53 K, SW54 J, SW55 U, SW56 SEITSEMÄN, SW57 GBP, SW58 DOUBLE_QUOTE, SW59 NOLLA, SW6 EQUALS, SW60 P, SW61 YHDEKSÄN, SW62 O, SW63 I, SW64 KAHDEKSAN, SW7 \BACKSLASH\, SW8 DELETE, SW9 SQUARE

Commit message: Swapped CAPS LOCK & DIAMOND
Parts:
- moved SW26 262.3 mm to (341.1, 187.7)
- moved SW33 262.3 mm to (81.6, 149.6)
Routing:
- net ROW3: track 332.3 -> 451.4 mm, vias 1 -> 2
- net ROW4: track 383.4 -> 296.2 mm, vias 1 -> 2
- net COL1: track 511.2 -> 573.8 mm, vias 1 -> 2
- net COL0: track 463.5 -> 449.2 mm
- net ROW7: track 230.8 -> 236.8 mm

Commit message: Finalised Rev. B design
Parts:
- removed G***: LOGO, LOGO
- removed KB4: SPACE_BAR, PCM_Mounting_Keyboard_Stabilizer:Stabilizer_Cherry_MX_7.00u
- added H3: MountingHole, MountingHole:MountingHole_3.2mm_M3, F.Cu at (250.7, 189.0)
- added H4: MountingHole, MountingHole:MountingHole_3.2mm_M3, F.Cu at (170.7, 189.0)
- added KB11: SPACE, PCM_Mounting_Keyboard_Stabilizer:Stabilizer_Cherry_MX_7.00u, F.Cu at (207.6, 187.7)
- SW12: value VASEN -> VASEN (L)
- SW13: value OIKEIN -> OIKEIN (R)
- SW14: value ALAS -> ALAS (D)
- SW15: value YLÖS -> YLÖS (U)
- SW19: value YKSI -> YKSI (1)
- SW20: value KAKSI -> KAKSI (2)
- SW21: value KOLME -> KOLME (3)
- SW22: value NELJÄ -> NELJÄ (4)
- SW23: value VIISI -> VIISI (5)
- SW24: value KUUSI -> KUUSI (6)
- SW41: value DOT -> .DOT.
- SW42: value COMMA -> ,COMMA,
- SW5: value UNDERSCORE -> _UNDERSCORE_
- SW50: value SEMICOLON -> ;SEMICOLON;
- SW56: value SEITSEMÄN -> SEITSEMÄN (7)
- SW59: value NOLLA -> NOLLA (0)
- SW6: value EQUALS -> =EQUALS=
- SW61: value YHDEKSÄN -> YHDEKSÄN (9)
- SW64: value KAHDEKSAN -> KAHDEKSAN (8)
- moved SK6 4.88 mm to (274.2, 100.1)
- moved SK7 4.84 mm to (300.1, 100.1)
Routing:
- net COL6: track 330.1 -> 317.6 mm, vias 2 -> 0
- net ROW7: track 236.8 -> 224.9 mm
- net ROW1: track 440.0 -> 430.1 mm
- net COL7: track 272.5 -> 266.8 mm
- net COL2: track 365.3 -> 360.3 mm
- net ROW5: track 464.1 -> 459.2 mm
- net COL1: track 573.8 -> 569.3 mm
- net ROW4: track 296.2 -> 293.0 mm, vias 2 -> 1
- net COL4: track 373.2 -> 370.0 mm
- net COL3: track 373.2 -> 370.0 mm
- net COL5: track 336.9 -> 333.8 mm
- net ROW2: track 271.3 -> 268.2 mm
- net ROW0: track 388.3 -> 385.3 mm
- net COL0: track 449.2 -> 446.4 mm
- net ROW6: track 254.9 -> 252.4 mm
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Other:
- outline, holes or cut-outs redrawn
- board text added: "(1.5u)"
- board text added: "(1.75u)"
- board text added: "(2u)"
- board text added: "(7u)"
- board text added: "(ISO)"
- board text removed: "1.5u"
- board text removed: "1.75u"
- board text removed: "2u"
- board text removed: "7u SPACE"
- board text removed: "ISO ENTER"
