File: Z88_Mechanical_Keyboard/Rev_B/Z88_Mechanical_Keyboard_Rev_B.kicad_sch (KiCad schematic)
At the start: 69 parts, among them SW1 SHIFT_RH, SW10 SHIFT_LH, SW11 SPACE, SW12 VASEN, SW13 OIKEIN, SW14 ALAS, SW15 YLÖS, SW16 ENTER, SW17 ESC, SW18 TAB, SW19 YKSI, SW2 APUA!, SW20 KAKSI, SW21 KOLME, SW22 NELJÄ, SW23 VIISI, SW24 KUUSI, SW25 INDEX, SW26 DIAMOND, SW27 Q, SW28 W, SW29 E, SW3 [, SW30 R, SW31 T, SW32 Y, SW33 CAPS_LOCK, SW34 MENU, SW35 A, SW36 S, SW37 D, SW38 F, SW39 G, SW4 ], SW40 H, SW41 DOT, SW42 COMMA, SW43 Z, SW44 X, SW45 C, SW46 V, SW47 B, SW48 N, SW49 /FORWSLASH/, SW5 UNDERSCORE, SW50 SEMICOLON, SW51 L, SW52 M, SW53 K, SW54 J, SW55 U, SW56 SEITSEMÄN, SW57 GBP, SW58 DOUBLE_QUOTE, SW59 NOLLA, SW6 EQUALS, SW60 P, SW61 YHDEKSÄN, SW62 O, SW63 I, SW64 KAHDEKSAN, SW7 \BACKSLASH\, SW8 DELETE, SW9 SQUARE

Commit message: Finalised Rev. B design
Parts:
- added H3, H4: MountingHole, MountingHole:MountingHole_3.2mm_M3, symbol Mechanical:MountingHole
- KB11: value SPACE_BAR -> SPACE
- SW12: value VASEN -> VASEN (L)
- SW13: value OIKEIN -> OIKEIN (R)
- SW14: value ALAS -> ALAS (D)
- SW15: value YLÖS -> YLÖS (U)
- SW19: value YKSI -> YKSI (1)
- SW20: value KAKSI -> KAKSI (2)
- SW21: value KOLME -> KOLME (3)
- SW22: value NELJÄ -> NELJÄ (4)
- SW23: value VIISI -> VIISI (5)
- SW24: value KUUSI -> KUUSI (6)
- SW41: value DOT -> .DOT.
- SW42: value COMMA -> ,COMMA,
- SW5: value UNDERSCORE -> _UNDERSCORE_
- SW50: value SEMICOLON -> ;SEMICOLON;
- SW56: value SEITSEMÄN -> SEITSEMÄN (7)
- SW59: value NOLLA -> NOLLA (0)
- SW6: value EQUALS -> =EQUALS=
- SW61: value YHDEKSÄN -> YHDEKSÄN (9)
- SW64: value KAHDEKSAN -> KAHDEKSAN (8)
Other:
- moved on the sheet: H1, H2
