File: Z88_Mechanical_Keyboard/ISO_Rev_B/Z88_Mechanical_Keyboard_Rev_B.kicad_pcb (KiCad board)
At the start: 2 copper layers, 289 x 110 mm, 68 parts, among them SW1 SHIFT_RH, SW10 SHIFT_LH, SW11 SPACE, SW12 LEFT, SW13 RIGHT, SW14 DOWN, SW15 UP, SW16 ENTER, SW17 ESC, SW18 TAB, SW19 ONE, SW2 HELP, SW20 2, SW21 3, SW22 4, SW23 5, SW24 6, SW25 INDEX, SW26 DIAMOND, SW27 Q, SW28 W, SW29 E, SW3 [, SW30 R, SW31 T, SW32 Y, SW33 CAPS_LOCK, SW34 MENU, SW35 A, SW36 S, SW37 D, SW38 F, SW39 G, SW4 ], SW40 H, SW41 DOT, SW42 COMMA, SW43 Z, SW44 X, SW45 C, SW46 V, SW47 B, SW48 N, SW49 /FORWSLASH/, SW5 UNDERSCORE, SW50 SEMICOLON, SW51 L, SW52 M, SW53 K, SW54 J, SW55 U, SW56 7, SW57 GBP, SW58 DOUBLE_QUOTE, SW59 ZERO, SW6 EQUALS, SW60 P, SW61 9, SW62 O, SW63 I, SW64 8, SW7 \BACKSLASH\, SW8 DELETE, SW9 SQUARE

Commit message: Updated ISO Rev. B, removed obsolete designs
Parts:
- added H3: MountingHole, MountingHole:MountingHole_3.2mm_M3, F.Cu at (250.7, 189.0)
- added H4: MountingHole, MountingHole:MountingHole_3.2mm_M3, F.Cu at (170.7, 185.0)
- added KB11: SPACE, PCM_Mounting_Keyboard_Stabilizer:Stabilizer_Cherry_MX_7.00u, F.Cu at (207.6, 187.7)
- SW12: value LEFT -> VASEN (L)
- SW13: value RIGHT -> OIKEIN (R)
- SW14: value DOWN -> ALAS (D)
- SW15: value UP -> YLÖS (U)
- SW19: value ONE -> YKSI (1)
- SW2: value HELP -> APUA!
- SW20: value 2 -> KAKSI (2)
- SW21: value 3 -> KOLME (3)
- SW22: value 4 -> NELJÄ (4)
- SW23: value 5 -> VIISI (5)
- SW24: value 6 -> KUUSI (6)
- SW41: value DOT -> .DOT.
- SW42: value COMMA -> ,COMMA,
- SW5: value UNDERSCORE -> _UNDERSCORE_
- SW50: value SEMICOLON -> ;SEMICOLON;
- SW56: value 7 -> SEITSEMÄN (7)
- SW59: value ZERO -> NOLLA (0)
- SW6: value EQUALS -> =EQUALS=
- SW61: value 9 -> YHDEKSÄN (9)
- SW64: value 8 -> KAHDEKSAN (8)
- moved SW26 262.3 mm to (341.1, 187.7)
- moved SW33 199.0 mm to (81.6, 149.6)
- moved SW14 38.1 mm to (303.0, 187.7)
- moved SW15 38.1 mm to (303.0, 168.7)
- moved H1 28.3 mm to (95.5, 97.0)
- moved SW1 19.1 mm to (331.7, 168.7)
- moved SW12 19.1 mm to (283.9, 187.7)
- moved H2 11.7 mm to (337.5, 97.0)
- moved SW11 6.93 mm to (207.6, 187.7)
- moved SK6 4.88 mm to (274.2, 100.1)
- moved SK7 4.84 mm to (300.1, 100.1)
- moved SW13 0.06 mm to (322.1, 187.7)
Routing:
- net COL1: track 0.00 -> 569.3 mm, vias 0 -> 2
- net ROW5: track 0.00 -> 459.2 mm, vias 0 -> 1
- net ROW3: track 0.00 -> 449.5 mm, vias 0 -> 2
- net COL0: track 0.00 -> 446.4 mm, vias 0 -> 1
- net ROW1: track 0.00 -> 430.1 mm
- net ROW0: track 0.00 -> 385.3 mm
- net COL4: track 0.00 -> 370.0 mm, vias 0 -> 2
- net COL3: track 0.00 -> 370.0 mm, vias 0 -> 2
- net COL2: track 0.00 -> 360.3 mm, vias 0 -> 1
- net COL5: track 0.00 -> 333.8 mm, vias 0 -> 1
- net COL6: track 0.00 -> 317.6 mm
- net ROW4: track 0.00 -> 293.0 mm, vias 0 -> 1
- net ROW2: track 0.00 -> 268.2 mm
- net COL7: track 0.00 -> 266.8 mm
- net ROW6: track 0.00 -> 252.4 mm, vias 0 -> 2
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Other:
- board size 289 x 110 mm -> 289 x 107.5 mm
- board text added: "(1.5u)"
- board text added: "(1.75u)"
- board text added: "(2u)"
- board text added: "(7u)"
- board text added: "(ISO)"
- board text added: "A14 A15 A13 A12 A11 A10 A9 A8"
- board text added: "Cambridge Computer Z88 Mechanical Keyboard Brett Hallen, Aug 2025 Port Macquarie, Australia WWW.YOUTUBE.COM/@BRFFF"
- board text added: "D5 D4 D3 D1 D7 D0 D6 D2"
- board text added: "Rev. B"
- board text added: "Sponsored by"
- board text added: "Z88мека"
- board text removed: "Cambridge Computer Z88"
- board text removed: "Cambridge Computer Z88 Mechanical Keyboard Brett Hallen, Jul 2025 Port Macquarie, Australia"
