File: Z88_Mechanical_Keyboard/ISO_Rev_B/Z88_Mechanical_Keyboard_ISO.kicad_pcb (KiCad board)
At the start: 2 copper layers, 289 x 107.5 mm, 71 parts, among them SW1 SHIFT_RH, SW10 SHIFT_LH, SW11 SPACE, SW12 VASEN (L), SW13 OIKEIN (R), SW14 ALAS (D), SW15 YLÖS (U), SW16 ENTER, SW17 ESC, SW18 TAB, SW19 YKSI (1), SW2 APUA!, SW20 KAKSI (2), SW21 KOLME (3), SW22 NELJÄ (4), SW23 VIISI (5), SW24 KUUSI (6), SW25 INDEX, SW26 DIAMOND, SW27 Q, SW28 W, SW29 E, SW3 [, SW30 R, SW31 T, SW32 Y, SW33 CAPS_LOCK, SW34 MENU, SW35 A, SW36 S, SW37 D, SW38 F, SW39 G, SW4 ], SW40 H, SW41 .DOT., SW42 ,COMMA,, SW43 Z, SW44 X, SW45 C, SW46 V, SW47 B, SW48 N, SW49 /FORWSLASH/, SW5 _UNDERSCORE_, SW50 ;SEMICOLON;, SW51 L, SW52 M, SW53 K, SW54 J, SW55 U, SW56 SEITSEMÄN (7), SW57 GBP, SW58 DOUBLE_QUOTE, SW59 NOLLA (0), SW6 =EQUALS=, SW60 P, SW61 YHDEKSÄN (9), SW62 O, SW63 I, SW64 KAHDEKSAN (8), SW7 \BACKSLASH\, SW8 DELETE, SW9 SQUARE

Commit message: Updated ISO layout keyboard
Other:
- board text added: "ISO Rev. B"
- board text removed: "Rev. B"
Changed lines of the file:
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@@
 	(paper "A3")
 	(title_block
-		(title "Z88 Mechanical Keyboard (Inverted-T Cursor)")
+		(title "Z88 Mechanical Keyboard (ISO Layout")
 		(date "16-Aug-2025")
 		(rev "B")
@@
 		)
 	)
-	(gr_text "Rev. B"
+	(gr_text "ISO\nRev. B"
 		(at 342.680241 97.5557 0)
 		(layer "F.SilkS")

Commit message: Cosmetic changes
Other:
- board text added: "Cambridge Computer Z88 Mechanical Keyboard Brett Hallen, Aug 2025 Port Macquarie, Australia www.youtube.com/@Brfff"
- board text added: "by Brett Hallen"
- board text removed: "Cambridge Computer Z88 Mechanical Keyboard Brett Hallen, Aug 2025 Port Macquarie, Australia WWW.YOUTUBE.COM/@BRFFF"
- board text removed: "Sponsored by"
