File: Z88_Mechanical_Keyboard/ANSI/Z88_Mechanical_Keyboard_ANSI.kicad_pcb (KiCad board)
At the start: 2 copper layers, 289 x 110 mm, 71 parts, among them SW1 SHIFT_RH, SW10 SHIFT_LH, SW11 SPACE, SW12 VASEN (L), SW13 OIKEIN (R), SW14 ALAS (D), SW15 YLÖS (U), SW16 ENTER, SW17 ESC, SW18 TAB, SW19 YKSI (1), SW2 APUA!, SW20 KAKSI (2), SW21 KOLME (3), SW22 NELJÄ (4), SW23 VIISI (5), SW24 KUUSI (6), SW25 INDEX, SW26 DIAMOND, SW27 Q, SW28 W, SW29 E, SW3 [, SW30 R, SW31 T, SW32 Y, SW33 CAPS_LOCK, SW34 MENU, SW35 A, SW36 S, SW37 D, SW38 F, SW39 G, SW4 ], SW40 H, SW41 .DOT., SW42 ,COMMA,, SW43 Z, SW44 X, SW45 C, SW46 V, SW47 B, SW48 N, SW49 /FORWSLASH/, SW5 _UNDERSCORE_, SW50 ;SEMICOLON;, SW51 L, SW52 M, SW53 K, SW54 J, SW55 U, SW56 SEITSEMÄN (7), SW57 GBP, SW58 DOUBLE_QUOTE, SW59 NOLLA (0), SW6 =EQUALS=, SW60 P, SW61 YHDEKSÄN (9), SW62 O, SW63 I, SW64 KAHDEKSAN (8), SW7 \BACKSLASH\, SW8 DELETE, SW9 SQUARE

Commit message: Updated ISO Rev. B, removed obsolete designs
Parts:
- moved SW57 38.3 mm to (321.8, 111.5)
- moved SW7 21.2 mm to (331.7, 130.4)
- moved SW16 19.2 mm to (322.1, 149.6)
Routing:
- net COL1: track 569.3 -> 0.00 mm, vias 2 -> 0
- net ROW5: track 459.2 -> 0.00 mm, vias 1 -> 0
- net ROW3: track 449.5 -> 0.00 mm, vias 2 -> 0
- net COL0: track 446.4 -> 0.00 mm, vias 1 -> 0
- net ROW1: track 430.1 -> 0.00 mm
- net ROW0: track 385.3 -> 0.00 mm
- net COL4: track 370.0 -> 0.00 mm, vias 2 -> 0
- net COL3: track 370.0 -> 0.00 mm, vias 2 -> 0
- net COL2: track 360.3 -> 0.00 mm, vias 1 -> 0
- net COL5: track 333.8 -> 0.00 mm, vias 1 -> 0
- net COL6: track 317.6 -> 0.00 mm
- net ROW4: track 293.0 -> 0.00 mm, vias 1 -> 0
- net ROW2: track 268.2 -> 0.00 mm
- net COL7: track 266.8 -> 0.00 mm
- net ROW6: track 252.4 -> 0.00 mm, vias 2 -> 0
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Other:
- board text removed: "(ISO)"

Commit message: ANSI keyboard design
Parts:
- moved SW16 7.12 mm to (329.3, 149.6)
- moved SW7 4.55 mm to (336.3, 130.5)
- moved H4 4.00 mm to (170.7, 185.0)
- moved SW57 0.32 mm to (322.1, 111.5)
Routing:
- net COL1: track 0.00 -> 569.3 mm, vias 0 -> 2
- net COL0: track 0.00 -> 465.3 mm
- net ROW1: track 0.00 -> 461.1 mm
- net ROW5: track 0.00 -> 459.2 mm, vias 0 -> 1
- net ROW3: track 0.00 -> 453.7 mm, vias 0 -> 2
- net ROW0: track 0.00 -> 386.4 mm
- net COL4: track 0.00 -> 370.0 mm, vias 0 -> 2
- net COL3: track 0.00 -> 370.0 mm, vias 0 -> 2
- net COL2: track 0.00 -> 360.3 mm, vias 0 -> 1
- net COL5: track 0.00 -> 333.8 mm, vias 0 -> 1
- net COL6: track 0.00 -> 331.3 mm
- net ROW4: track 0.00 -> 293.0 mm, vias 0 -> 1
- net COL7: track 0.00 -> 280.4 mm
- net ROW2: track 0.00 -> 268.2 mm
- net ROW6: track 0.00 -> 252.4 mm, vias 0 -> 2
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Other:
- board size 289 x 110 mm -> 289 x 107.5 mm
- board text added: "(2.25u)"
- board text added: "ANSI Rev. B"
- board text added: "Cambridge Computer Z88 Mechanical Keyboard Brett Hallen, Aug 2025 Port Macquarie, Australia WWW.YOUTUBE.COM/@BRFFF"
- board text added: "Z88мека"
- board text removed: "Cambridge Computer Z88"
- board text removed: "Cambridge Computer Z88 Mechanical Keyboard Brett Hallen, Jul 2025 Port Macquarie, Australia WWW.YOUTUBE.COM/@BRFFF"
- board text removed: "Rev. B"

Commit message: Cosmetic changes
Other:
- board text added: "Cambridge Computer Z88 Mechanical Keyboard Brett Hallen, Aug 2025 Port Macquarie, Australia www.youtube.com/@Brfff"
- board text added: "by Brett Hallen"
- board text removed: "Cambridge Computer Z88 Mechanical Keyboard Brett Hallen, Aug 2025 Port Macquarie, Australia WWW.YOUTUBE.COM/@BRFFF"
- board text removed: "Sponsored by"
